Commit message: Localizer rejects vlam poses if markers are too far away

File: orca_description/xacro/orca.urdf.xacro (robot description, xacro)
@@ -39,5 +39,5 @@
     <!-- Sensor properties -->
     <xacro:property name="BARO_FREQ" value="20.0"/>
-    <xacro:property name="CAMERA_FREQ" value="10.0"/>
+    <xacro:property name="CAMERA_FREQ" value="1.0"/>
     <!-- General constants -->
     <xacro:property name="PI" value="3.1415926535897931"/>
@@ -424,20 +424,20 @@
     </xacro:macro>
     <!-- Forward-facing camera: -->
-    <xacro:camera_plugin prefix="forward" width="800" height="600" horizontal_fov="1.4"/>
+    <xacro:camera_plugin prefix="forward" width="1920" height="1080" horizontal_fov="1.4"/>
     <!-- Left down-facing camera: -->
 <!--    <xacro:camera_plugin prefix="left" width="800" height="600" horizontal_fov="1.4"/>-->
     <!-- Right down-facing camera: -->
 <!--    <xacro:camera_plugin prefix="right" width="800" height="600" horizontal_fov="1.4"/>-->
-    <gazebo>
-        <plugin name="p3d_test" filename="libgazebo_ros_p3d.so">
-            <ros>
-                <argument>odom:=ground_truth</argument>
-            </ros>
-            <update_rate>30.0</update_rate>
-            <body_name>base_link</body_name>
-            <frame_name>map</frame_name>
-            <xyz_offsets>0 0 0</xyz_offsets>
-            <rpy_offsets>0 0 0</rpy_offsets>
-        </plugin>
-    </gazebo>
+<!--    <gazebo>-->
+<!--        <plugin name="p3d_test" filename="libgazebo_ros_p3d.so">-->
+<!--            <ros>-->
+<!--                <argument>odom:=ground_truth</argument>-->
+<!--            </ros>-->
+<!--            <update_rate>30.0</update_rate>-->
+<!--            <body_name>base_link</body_name>-->
+<!--            <frame_name>map</frame_name>-->
+<!--            <xyz_offsets>0 0 0</xyz_offsets>-->
+<!--            <rpy_offsets>0 0 0</rpy_offsets>-->
+<!--        </plugin>-->
+<!--    </gazebo>-->
 </robot>

Commit message: Harmonize, cleanup Gazebo plugins

File: orca_description/xacro/orca.urdf.xacro (robot description, xacro)
@@ -298,9 +298,8 @@
     <gazebo>
         <plugin name="OrcaBuoyancyPlugin" filename="libOrcaBuoyancyPlugin.so">
+            <base_link>base_link</base_link>
+            <center_of_volume>0 0 ${VOLUME_Z}</center_of_volume>
             <fluid_density>${FLUID_DENSITY}</fluid_density>
-            <link name="base_link">
-                <center_of_volume>0 0 ${VOLUME_Z}</center_of_volume>
-                <volume>${TOTAL_VOLUME}</volume>
-            </link>
+            <volume>${TOTAL_VOLUME}</volume>
         </plugin>
     </gazebo>
@@ -310,9 +309,7 @@
     <gazebo>
         <plugin name="OrcaDragPlugin" filename="libOrcaDragPlugin.so">
-            <link name="base_link">
-                <center_of_mass>0 0 ${MASS_Z}</center_of_mass>
-                <center_of_volume>0 0 ${VOLUME_Z}</center_of_volume>
-                <angular_drag>4 4 4</angular_drag>
-            </link>
+            <angular_drag>4 4 4</angular_drag>
+            <base_link>base_link</base_link>
+            <center_of_mass>0 0 ${MASS_Z}</center_of_mass>
         </plugin>
     </gazebo>
@@ -323,5 +320,5 @@
     <gazebo>
         <plugin name="OrcaThrusterPlugin" filename="libOrcaThrusterPlugin.so">
-            <link_name>orca::base_link</link_name>
+            <base_link>base_link</base_link>
             <thruster name="front_right"> <!-- name attributes are ignored; the tag order must match the message array order -->
                 <pos_force>${FORWARD_FORCE}</pos_force> <!-- units are N, positive for ccw, negative for cw -->

Commit message: First cut at README files

File: orca_description/xacro/orca.urdf.xacro (robot description, xacro)
@@ -39,4 +39,5 @@
     <!-- Sensor properties -->
     <xacro:property name="BARO_FREQ" value="20.0"/>
+    <xacro:property name="BARO_VAR" value="40682.89"/>
     <xacro:property name="CAMERA_FREQ" value="1.0"/>
     <!-- General constants -->
@@ -361,4 +362,6 @@
             <plugin name="OrcaBarometerPlugin" filename="libOrcaBarometerPlugin.so">
                 <fluid_density>${FLUID_DENSITY}</fluid_density>
+                <baro_link_to_base_link_z_>0.05</baro_link_to_base_link_z_>
+                <variance>${BARO_VAR}</variance>
             </plugin>
         </sensor>

Commit message: Reformat

File: orca_description/xacro/orca.urdf.xacro (robot description, xacro)
@@ -1,432 +1,426 @@
 <?xml version="1.0"?>
 <robot name="orca" xmlns:xacro="http://ros.org/wiki/xacro">
-    <!--
-        Orca constants
-        Flight dynamics are hugely driven by these 3 constants, all in the body frame:
-            {x, y, THRUSTER_Z}: where forward/back/strafe/yaw thrust forces are applied
-            {0, 0, MASS_Z}: where the linear and angular drag force is applied
-            {0, 0, VOLUME_Z}: where the buoyancy force is applied
-        Default simulation is fresh water and slightly positive buoyancy:
-            TOTAL_VOLUME = 0.01
-            FLUID_DENSITY = 997
-            DISPLACED_MASS = TOTAL_VOLUME * FLUID_DENSITY = 9.97
-            TOTAL_MASS = 9.9
-     -->
-    <xacro:property name="TOTAL_MASS" value="9.9"/>
-    <xacro:property name="TOTAL_VOLUME" value="0.01"/>
-    <xacro:property name="LENGTH" value="0.457"/>
-    <xacro:property name="WIDTH" value="0.338"/>
-    <xacro:property name="HEIGHT" value="0.25"/>
-    <xacro:property name="IXX" value="${TOTAL_MASS / 12 * (WIDTH * WIDTH + HEIGHT * HEIGHT)}"/>
-    <xacro:property name="IYY" value="${TOTAL_MASS / 12 * (LENGTH * LENGTH + HEIGHT * HEIGHT)}"/>
-    <xacro:property name="IZZ" value="${TOTAL_MASS / 12 * (LENGTH * LENGTH + WIDTH * WIDTH)}"/>
-    <xacro:property name="FLOAT_X" value="0.12"/>
-    <xacro:property name="FLOAT_Y" value="0.11"/>
-    <xacro:property name="FLOAT_Z" value="0.07"/>
-    <xacro:property name="THRUSTER_X" value="0.15"/>
-    <xacro:property name="THRUSTER_Y" value="0.09"/>
-    <xacro:property name="THRUSTER_Z" value="-0.009"/>
-    <xacro:property name="VERT_THRUSTER_Y" value="0.105"/>
-    <xacro:property name="VERT_THRUSTER_Z" value="0.09"/>
-    <xacro:property name="MASS_Z" value="0.011"/>
-    <xacro:property name="VOLUME_Z" value="0.06"/>
-    <xacro:property name="FORWARD_FORCE" value="50"/>
-    <xacro:property name="REVERSE_FORCE" value="40"/>
-    <xacro:property name="HAS_TETHER" default="false"/>
-    <xacro:property name="SURFACE" default="0"/>
-    <!-- Physics properties -->
-    <xacro:property name="FLUID_DENSITY" value="997"/>
-    <!-- Sensor properties -->
-    <xacro:property name="BARO_FREQ" value="20.0"/>
-    <xacro:property name="BARO_VAR" value="40682.89"/>
-    <xacro:property name="CAMERA_FREQ" value="1.0"/>
-    <!-- General constants -->
-    <xacro:property name="PI" value="3.1415926535897931"/>
-    <!-- Materials -->
-    <material name="gray">
-        <color rgba="0.5 0.5 0.5 1.0"/>
-    </material>
-    <material name="blue">
-        <color rgba="0.5 0.5 1.0 1.0"/>
-    </material>
-    <material name="red">
-        <color rgba="1.0 0.0 0.0 1.0"/>
-    </material>
-    <!-- Thruster origins -->
-    <xacro:property name="front_right_origin">
-        <origin xyz="${THRUSTER_X} ${-THRUSTER_Y} ${THRUSTER_Z}" rpy="0 ${PI/2} ${PI/4}"/>
-    </xacro:property>
-    <xacro:property name="front_left_origin">
-        <origin xyz="${THRUSTER_X} ${THRUSTER_Y} ${THRUSTER_Z}" rpy="0 ${PI/2} ${-PI/4}"/>
-    </xacro:property>
-    <xacro:property name="rear_right_origin">
-        <origin xyz="${-THRUSTER_X} ${-THRUSTER_Y} ${THRUSTER_Z}" rpy="0 ${PI/2} ${PI*3/4}"/>
-    </xacro:property>
-    <xacro:property name="rear_left_origin">
-        <origin xyz="${-THRUSTER_X} ${THRUSTER_Y} ${THRUSTER_Z}" rpy="0 ${PI/2} ${-PI*3/4}"/>
-    </xacro:property>
-    <xacro:property name="vertical_right_origin">
-        <origin xyz="0 ${-VERT_THRUSTER_Y} ${VERT_THRUSTER_Z}" rpy="0 0 0"/>
-    </xacro:property>
-    <xacro:property name="vertical_left_origin">
-        <origin xyz="0 ${VERT_THRUSTER_Y} ${VERT_THRUSTER_Z}" rpy="0 0 0"/>
-    </xacro:property>
-    <!-- Thruster macro -->
-    <xacro:macro name="t200" params="name *origin">
-        <link name="t200_link_${name}">
-            <!-- Front cone -->
-            <visual>
-                <origin xyz="0 0 0"/>
-                <geometry>
-                    <sphere radius="0.02"/>
-                </geometry>
-                <material name="gray"/> <!-- All visual elements in this link pick up this material -->
-            </visual>
-            <!-- Rear cone -->
-            <visual>
-                <origin xyz="0 0 -0.07"/>
-                <geometry>
-                    <sphere radius="0.02"/>
-                </geometry>
-            </visual>
-            <!-- Thruster body -->
-            <visual>
-                <origin xyz="0 0 -0.035"/>
-                <geometry>
-                    <cylinder length="0.07" radius="0.02"/>
-                </geometry>
-            </visual>
-            <!-- Propeller guard -->
-            <visual>
-                <origin xyz="0 0 -0.0225"/>
-                <geometry>
-                    <cylinder length="0.045" radius="0.045"/>
-                </geometry>
-            </visual>
-        </link>
-        <joint name="t200_joint_${name}" type="fixed">
-            <xacro:insert_block name="origin"/>
-            <parent link="base_link"/>
-            <child link="t200_link_${name}"/>
-        </joint>
-    </xacro:macro>
-    <!-- Base link -->
-    <link name="base_link">
-        <!-- Inertial -->
-        <inertial>
-            <origin xyz="0 0 ${MASS_Z}"/> <!-- Center of mass -->
-            <mass value="${TOTAL_MASS}"/>
-            <inertia ixx="${IXX}" ixy="0.0" ixz="0.0" iyy="${IYY}" iyz="0.0" izz="${IZZ}"/>
-        </inertial>
-        <!-- Float -->
-        <visual>
-            <origin xyz="${FLOAT_X} ${FLOAT_Y} ${FLOAT_Z}"/>
-            <geometry>
-                <box size="0.15 0.09 0.08"/>
-            </geometry>
-            <material name="blue"/>
-        </visual>
-        <!-- Float -->
-        <visual>
-            <origin xyz="${FLOAT_X} ${-FLOAT_Y} ${FLOAT_Z}"/>
-            <geometry>
-                <box size="0.15 0.09 0.08"/>
-            </geometry>
-        </visual>
-        <!-- Float -->
-        <visual>
-            <origin xyz="${-FLOAT_X} ${FLOAT_Y} ${FLOAT_Z}"/>
-            <geometry>
-                <box size="0.15 0.09 0.08"/>
-            </geometry>
-        </visual>
-        <!-- Float -->
-        <visual>
-            <origin xyz="${-FLOAT_X} ${-FLOAT_Y} ${FLOAT_Z}"/>
-            <geometry>
-                <box size="0.15 0.09 0.08"/>
-            </geometry>
-        </visual>
-        <!-- Electronics tube -->
-        <visual>
-            <origin xyz="0 0 0.063" rpy="0 ${PI/2} 0"/>
-            <geometry>
-                <cylinder length="0.32" radius="0.055"/>
-            </geometry>
-        </visual>
-        <!-- Battery tube -->
-        <visual>
-            <origin xyz="0 0 -0.05" rpy="0 ${PI/2} 0"/>
-            <geometry>
-                <cylinder length="0.25" radius="0.045"/>
-            </geometry>
-        </visual>
-        <!-- Left down-facing camera tube -->
-        <visual>
-            <origin xyz="-0.15 0.18 0" rpy="0 0 0"/>
-            <geometry>
-                <cylinder length="0.135" radius="0.0275"/>
-            </geometry>
-        </visual>
-        <!-- Right down-facing camera tube -->
-        <visual>
-            <origin xyz="-0.15 -0.18 0" rpy="0 0 0"/>
-            <geometry>
-                <cylinder length="0.135" radius="0.0275"/>
-            </geometry>
-        </visual>
-        <!-- Collision region -->
-        <collision>
-            <geometry>
-                <box size="${LENGTH} ${WIDTH} ${HEIGHT}"/>
-            </geometry>
-        </collision>
+  <!--
+      Orca constants
+      Flight dynamics are hugely driven by these 3 constants, all in the body frame:
+          {x, y, THRUSTER_Z}: where forward/back/strafe/yaw thrust forces are applied
+          {0, 0, MASS_Z}: where the linear and angular drag force is applied
+          {0, 0, VOLUME_Z}: where the buoyancy force is applied
+      Default simulation is fresh water and slightly positive buoyancy:
+          TOTAL_VOLUME = 0.01
+          FLUID_DENSITY = 997
+          DISPLACED_MASS = TOTAL_VOLUME * FLUID_DENSITY = 9.97
+          TOTAL_MASS = 9.9
+   -->
+  <xacro:property name="TOTAL_MASS" value="9.9"/>
+  <xacro:property name="TOTAL_VOLUME" value="0.01"/>
+  <xacro:property name="LENGTH" value="0.457"/>
+  <xacro:property name="WIDTH" value="0.338"/>
+  <xacro:property name="HEIGHT" value="0.25"/>
+  <xacro:property name="IXX" value="${TOTAL_MASS / 12 * (WIDTH * WIDTH + HEIGHT * HEIGHT)}"/>
+  <xacro:property name="IYY" value="${TOTAL_MASS / 12 * (LENGTH * LENGTH + HEIGHT * HEIGHT)}"/>
+  <xacro:property name="IZZ" value="${TOTAL_MASS / 12 * (LENGTH * LENGTH + WIDTH * WIDTH)}"/>
+  <xacro:property name="FLOAT_X" value="0.12"/>
+  <xacro:property name="FLOAT_Y" value="0.11"/>
+  <xacro:property name="FLOAT_Z" value="0.07"/>
+  <xacro:property name="THRUSTER_X" value="0.15"/>
+  <xacro:property name="THRUSTER_Y" value="0.09"/>
+  <xacro:property name="THRUSTER_Z" value="-0.009"/>
+  <xacro:property name="VERT_THRUSTER_Y" value="0.105"/>
+  <xacro:property name="VERT_THRUSTER_Z" value="0.09"/>
+  <xacro:property name="MASS_Z" value="0.011"/>
+  <xacro:property name="VOLUME_Z" value="0.06"/>
+  <xacro:property name="FORWARD_FORCE" value="50"/>
+  <xacro:property name="REVERSE_FORCE" value="40"/>
+  <xacro:property name="HAS_TETHER" default="false"/>
+  <xacro:property name="SURFACE" default="0"/>
+  <!-- Physics properties -->
+  <xacro:property name="FLUID_DENSITY" value="997"/>
+  <!-- Sensor properties -->
+  <xacro:property name="BARO_FREQ" value="20.0"/>
+  <xacro:property name="BARO_VAR" value="40682.89"/>
+  <xacro:property name="CAMERA_FREQ" value="1.0"/>
+  <!-- General constants -->
+  <xacro:property name="PI" value="3.1415926535897931"/>
+  <!-- Materials -->
+  <material name="gray">
+    <color rgba="0.5 0.5 0.5 1.0"/>
+  </material>
+  <material name="blue">
+    <color rgba="0.5 0.5 1.0 1.0"/>
+  </material>
+  <material name="red">
+    <color rgba="1.0 0.0 0.0 1.0"/>
+  </material>
+  <!-- Thruster origins -->
+  <xacro:property name="front_right_origin">
+    <origin xyz="${THRUSTER_X} ${-THRUSTER_Y} ${THRUSTER_Z}" rpy="0 ${PI/2} ${PI/4}"/>
+  </xacro:property>
+  <xacro:property name="front_left_origin">
+    <origin xyz="${THRUSTER_X} ${THRUSTER_Y} ${THRUSTER_Z}" rpy="0 ${PI/2} ${-PI/4}"/>
+  </xacro:property>
+  <xacro:property name="rear_right_origin">
+    <origin xyz="${-THRUSTER_X} ${-THRUSTER_Y} ${THRUSTER_Z}" rpy="0 ${PI/2} ${PI*3/4}"/>
+  </xacro:property>
+  <xacro:property name="rear_left_origin">
+    <origin xyz="${-THRUSTER_X} ${THRUSTER_Y} ${THRUSTER_Z}" rpy="0 ${PI/2} ${-PI*3/4}"/>
+  </xacro:property>
+  <xacro:property name="vertical_right_origin">
+    <origin xyz="0 ${-VERT_THRUSTER_Y} ${VERT_THRUSTER_Z}" rpy="0 0 0"/>
+  </xacro:property>
+  <xacro:property name="vertical_left_origin">
+    <origin xyz="0 ${VERT_THRUSTER_Y} ${VERT_THRUSTER_Z}" rpy="0 0 0"/>
+  </xacro:property>
+  <!-- Thruster macro -->
+  <xacro:macro name="t200" params="name *origin">
+    <link name="t200_link_${name}">
+      <!-- Front cone -->
+      <visual>
+        <origin xyz="0 0 0"/>
+        <geometry>
+          <sphere radius="0.02"/>
+        </geometry>
+        <material name="gray"/> <!-- All visual elements in this link pick up this material -->
+      </visual>
+      <!-- Rear cone -->
+      <visual>
+        <origin xyz="0 0 -0.07"/>
+        <geometry>
+          <sphere radius="0.02"/>
+        </geometry>
+      </visual>
+      <!-- Thruster body -->
+      <visual>
+        <origin xyz="0 0 -0.035"/>
+        <geometry>
+          <cylinder length="0.07" radius="0.02"/>
+        </geometry>
+      </visual>
+      <!-- Propeller guard -->
+      <visual>
+        <origin xyz="0 0 -0.0225"/>
+        <geometry>
+          <cylinder length="0.045" radius="0.045"/>
+        </geometry>
+      </visual>
     </link>
-    <!-- Barometer link -->
-    <link name="baro_link">
-        <visual>
-            <origin xyz="0 0 0" rpy="0 ${PI/2} 0"/>
-            <geometry>
-                <cylinder length="0.01" radius="0.01"/>
-            </geometry>
-            <material name="red"/>
-        </visual>
-    </link>
-    <!-- Attach baro_link to base_link -->
-    <joint name="baro_joint" type="fixed">
-        <origin xyz="-0.16 0 0.05" rpy="0 0 0"/>
-        <parent link="base_link"/>
-        <child link="baro_link"/>
+    <joint name="t200_joint_${name}" type="fixed">
+      <xacro:insert_block name="origin"/>
+      <parent link="base_link"/>
+      <child link="t200_link_${name}"/>
     </joint>
-    <!-- Forward camera link -->
-    <link name="forward_camera_link">
-        <visual>
-            <origin xyz="0 0 0" rpy="0 0 0"/>
-            <geometry>
-                <sphere radius="0.052"/>
-            </geometry>
-            <material name="red"/>
-        </visual>
-    </link>
-    <!-- Attach forward_camera_link to base_link -->
-    <joint name="forward_camera_joint" type="fixed">
-        <origin xyz="0.16 0 0.063" rpy="0 0 0"/>
-        <parent link="base_link"/>
-        <child link="forward_camera_link"/>
-    </joint>
-    <!-- Forward camera frame -->
-    <link name="forward_camera_frame"/>
-    <!-- Attach forward_camera_frame to base_link (parsed by filter_node) -->
-    <joint name="forward_camera_frame_joint" type="fixed">
-        <origin xyz="0.16 0 0.063" rpy="${-PI/2} 0 ${-PI/2}"/>
-        <parent link="base_link"/>
-        <child link="forward_camera_frame"/>
-    </joint>
-    <!-- Left and right cameras are positioned to see markers along the seafloor. Both are portrait. -->
-    <!-- Left camera link -->
-    <link name="left_camera_link">
-        <visual>
-            <origin xyz="0 0 0" rpy="0 0 0"/>
-            <geometry>
-                <!-- Make the aspect ratio obvious -->
-                <box size="0.01 0.04 0.03"/>
-            </geometry>
-            <material name="red"/>
-        </visual>
-    </link>
-    <!-- Attach left_camera_link to base_link -->
-    <joint name="left_camera_joint" type="fixed">
-        <origin xyz="-0.15 0.18 -0.0675" rpy="${PI/2} ${PI/2} 0"/>
-        <parent link="base_link"/>
-        <child link="left_camera_link"/>
-    </joint>
-    <!-- Left camera frame -->
-    <link name="left_camera_frame"/>
-    <!-- Attach left_camera_frame to base_link (parsed by filter_node)  -->
-    <joint name="left_camera_frame_joint" type="fixed">
-        <origin xyz="-0.15 0.18 -0.0675" rpy="0 ${PI} 0"/>
-        <parent link="base_link"/>
-        <child link="left_camera_frame"/>
-    </joint>
-    <!-- Right camera link -->
-    <link name="right_camera_link">
-        <visual>
-            <origin xyz="0 0 0" rpy="0 0 0"/>
-            <geometry>
-                <!-- Make the aspect ratio obvious -->
-                <box size="0.01 0.04 0.03"/>
-            </geometry>
-            <material name="red"/>
-        </visual>
-    </link>
-    <!-- Attach right_camera_link to base_link -->
-    <joint name="right_camera_joint" type="fixed">
-        <origin xyz="-0.15 -0.18 -0.0675" rpy="${PI/2} ${PI/2} 0"/>
-        <parent link="base_link"/>
-        <child link="right_camera_link"/>
-    </joint>
-    <!-- Right camera frame -->
-    <link name="right_camera_frame"/>
-    <!-- Attach right_camera_frame to base_link (parsed by filter_node) -->
-    <joint name="right_camera_frame_joint" type="fixed">
-        <origin xyz="-0.15 -0.18 -0.0675" rpy="0 ${PI} 0"/>
-        <parent link="base_link"/>
-        <child link="right_camera_frame"/>
-    </joint>
-    <!-- Attach thrusters to the base_link -->
-    <xacro:t200 name="front_right">
+  </xacro:macro>
+  <!-- Base link -->
+  <link name="base_link">
+    <!-- Inertial -->
+    <inertial>
+      <origin xyz="0 0 ${MASS_Z}"/> <!-- Center of mass -->
+      <mass value="${TOTAL_MASS}"/>
+      <inertia ixx="${IXX}" ixy="0.0" ixz="0.0" iyy="${IYY}" iyz="0.0" izz="${IZZ}"/>
+    </inertial>
+    <!-- Float -->
+    <visual>
+      <origin xyz="${FLOAT_X} ${FLOAT_Y} ${FLOAT_Z}"/>
+      <geometry>
+        <box size="0.15 0.09 0.08"/>
+      </geometry>
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