Commit message: Checkpoint: testing stereo rig

File: orca_description/xacro/orca.urdf.xacro (robot description, xacro)
@@ -48,7 +48,7 @@
   <xacro:property name="FORWARD_FORCE" value="50"/>
   <xacro:property name="REVERSE_FORCE" value="40"/>
-  <xacro:property name="HAS_TETHER" default="false"/>
-  <xacro:property name="SURFACE" default="0"/>
-  <xacro:property name="STEREO_BASELINE" default="0.36"/>
+  <xacro:property name="HAS_TETHER" value="false"/>
+  <xacro:property name="SURFACE" value="0"/>
+  <xacro:property name="STEREO_BASELINE" value="0.36"/>
   <!-- Physics properties -->
   <xacro:property name="FLUID_DENSITY" value="997"/>

Commit message: Add camera distortion to slam test

File: orca_description/xacro/orca.urdf.xacro (robot description, xacro)
@@ -16,4 +16,6 @@
   <xacro:property name="MOTION_PLUGIN" value="${SIM_MODE == 'slam_test'}"/>
   <xacro:property name="GROUND_TRUTH_PLUGIN" value="true"/>
+  <!-- Enable distortion on the stereo camera for the slam test -->
+  <xacro:property name="STEREO_DISTORTION" value="${SIM_MODE == 'slam_test'}"/>
   <!--
       Orca constants
@@ -456,4 +458,18 @@
             <far>${CAMERA_FAR_CLIP}</far>
           </clip>
+          <xacro:if value="${STEREO_DISTORTION}">
+            <!-- Simulate some barrel distortion to test the image pipeline.
+                 Be sure to set border_crop=False below. If the border is cropped
+                 image_proc::RectifyNode will not correctly rectify the image.
+                 Note that the rectification matrix camera_info.r is always the identity matrix.
+                 See gazebo_plugins/src/gazebo_ros_camera.cpp for details. -->
+            <distortion>
+              <k1>-0.25</k1>
+              <k2>0.12</k2>
+              <p1>-0.00028</p1>
+              <p2>-0.00005</p2>
+              <k3>0.0</k3>
+            </distortion>
+          </xacro:if>
           <noise>
             <type>gaussian</type>
@@ -477,4 +493,13 @@
             <far>${CAMERA_FAR_CLIP}</far>
           </clip>
+          <xacro:if value="${STEREO_DISTORTION}">
+            <distortion>
+              <k1>-0.25</k1>
+              <k2>0.12</k2>
+              <p1>-0.00028</p1>
+              <p2>-0.00005</p2>
+              <k3>0.0</k3>
+            </distortion>
+          </xacro:if>
           <noise>
             <type>gaussian</type>
@@ -490,5 +515,5 @@
           <!-- Default frame name is the link name (left_camera_link). Override to distinguish
                between the link, which pitches forward pi/4, and the camera frame, which pitches
-               forward pi/2. Both cameras will use the same frame name -->
+               forward pi/2. Both cameras will use the same frame name. -->
           <frame_name>left_camera_frame</frame_name>
           <!-- The baseline value is the distance between the 2 cameras. It shows up in the
@@ -497,4 +522,7 @@
                hack_baseline tag. -->
           <hack_baseline>${STEREO_BASELINE}</hack_baseline>
+          <!-- Turn off border cropping so that downstream nodes can use the provided distortion
+               values to restore the image. -->
+          <border_crop>False</border_crop>
         </plugin>
       </sensor>

Commit message: TeleopNode can launch video pipelines without UI

File: orca_description/xacro/orca.urdf.xacro (robot description, xacro)
@@ -59,5 +59,5 @@
   <xacro:property name="BARO_VAR" value="40682.89"/>
   <xacro:property name="FWD_CAMERA_FREQ" value="1.0"/> <!-- Hack: slow down updates -->
-  <xacro:property name="DOWN_CAMERA_FREQ" value="30.0"/>
+  <xacro:property name="DOWN_CAMERA_FREQ" value="20.0"/>
   <xacro:property name="CAMERA_STD_DEV" value="0.07"/>
   <xacro:property name="CAMERA_FAR_CLIP" value="10"/>
